File: CapSensors.kicad_sch (KiCad schematic)
At the start: 6 parts, among them J1 Charge/Discharge Pins, J2 Analog Pins, J3 Ground, J4 Charge/Discharge Pins

Commit message: Add files via upload
Parts:
- removed J1, J4: Charge/Discharge Pins, TerminalBlock_4Ucon:TerminalBlock_4Ucon_1x15_P3.50mm_Vertical, symbol Connector:Conn_01x15_Female
- removed J2: Analog Pins, TerminalBlock_4Ucon:TerminalBlock_4Ucon_1x15_P3.50mm_Vertical, symbol Connector:Conn_01x15_Female
- removed J3: Ground, TerminalBlock_4Ucon:TerminalBlock_4Ucon_1x15_P3.50mm_Vertical, symbol Connector:Conn_01x15_Female
- added AnalogPins1, Ground1: Screw_Terminal_01x15, TerminalBlock_TE-Connectivity:TerminalBlock_TE_1-282834-2_1x12_P2.54mm_Horizontal, symbol Connector:Screw_Terminal_01x15
- added ChargePins1, DischargePins1: Conn_01x15_Male, Connector_PinHeader_2.54mm:PinHeader_1x15_P2.54mm_Vertical, symbol Connector:Conn_01x15_Male
- added R10, R13, R15, R17, R19, R21, R23, R25, R27, R29, R3, R4, R6, R8: 10k, Resistor_SMD:R_0603_1608Metric, symbol Device:R
- added R11, R12, R14, R16, R18, R20, R22, R24, R26, R28, R30, R5, R7, R9: 220, Resistor_SMD:R_0603_1608Metric, symbol Device:R
Connections:
- net C1 charge: now also ChargePins1.1 (Pin_1)
- net C1 discharge: now also DischargePins1.1 (Pin_1)
- net GND: now also Ground1.1 (Pin_1), Ground1.10 (Pin_10), Ground1.11 (Pin_11), Ground1.12 (Pin_12), Ground1.13 (Pin_13), Ground1.14 (Pin_14), Ground1.15 (Pin_15), Ground1.2 (Pin_2), Ground1.3 (Pin_3), Ground1.4 (Pin_4), Ground1.5 (Pin_5), Ground1.6 (Pin_6), Ground1.7 (Pin_7), Ground1.8 (Pin_8), Ground1.9 (Pin_9)
- net Analog1: now reaches R1.2, R2.1
- net Analog1: now also AnalogPins1.1 (Pin_1)
- new net Analog10: AnalogPins1.10 (Pin_10), R19.2, R20.1
- new net Analog11: AnalogPins1.11 (Pin_11), R21.2, R22.1
- new net Analog12: AnalogPins1.12 (Pin_12), R23.2, R24.1
- new net Analog13: AnalogPins1.13 (Pin_13), R25.2, R26.1
- new net Analog14: AnalogPins1.14 (Pin_14), R27.2, R28.1
- new net Analog15: AnalogPins1.15 (Pin_15), R29.2, R30.1
- new net Analog2: AnalogPins1.2 (Pin_2), R12.1, R3.2
- new net Analog3: AnalogPins1.3 (Pin_3), R6.2, R7.1
- new net Analog4: AnalogPins1.4 (Pin_4), R8.2, R9.1
- new net Analog5: AnalogPins1.5 (Pin_5), R10.2, R11.1
- new net Analog6: AnalogPins1.6 (Pin_6), R4.2, R5.1
- new net Analog7: AnalogPins1.7 (Pin_7), R13.2, R14.1
- new net Analog8: AnalogPins1.8 (Pin_8), R15.2, R16.1
- new net Analog9: AnalogPins1.9 (Pin_9), R17.2, R18.1
- new net C10 charge: R19.1
- new net C10 discharge: R20.2
- new net C11 charge: R21.1
- new net C11 discharge: R22.2
- new net C12 charge: R23.1
- new net C12 discharge: R24.2
- new net C13 charge: R25.1
- new net C13 discharge: R26.2
- new net C14 charge: R27.1
- new net C14 discharge: R28.2
- new net C15 charge: R29.1
- new net C15 discharge: R30.2
- new net C2 charge: R3.1
- new net C2 discharge: R12.2
- new net C3 charge: R6.1
- new net C3 discharge: R7.2
- new net C4 charge: R8.1
- new net C4 discharge: R9.2
- new net C5 charge: R10.1
- new net C5 discharge: R11.2
- new net C6 charge: R4.1
- new net C6 discharge: R5.2
- new net C7 charge: R13.1
- new net C7 discharge: R14.2
- new net C8 charge: R15.1
- new net C8 discharge: R16.2
- new net C9 charge: R17.1
- new net C9 discharge: R18.2
