File: CapSensors.kicad_sch (KiCad schematic)
At the start: 34 parts

Commit message: Add files via upload
Parts:
- removed DischargePins1: Conn_01x15_Female, Connector_PinHeader_2.54mm:PinHeader_1x15_P2.54mm_Vertical, symbol Connector:Conn_01x15_Female
- added Charge/DischargePins2: Conn_01x15_Female, Connector_PinHeader_2.54mm:PinHeader_1x15_P2.54mm_Vertical, symbol Connector:Conn_01x15_Female
- added Ground: Conn_01x01_Female, Connector_PinHeader_2.54mm:PinHeader_1x01_P2.54mm_Vertical, symbol Connector:Conn_01x01_Female
- renumbered AnalogPins1 to Analog/GroundPins1, Ground1 to Analog/GroundPins2, ChargePins1 to Charge/DischargePins1, R11 to R10, R4 to R11, R5 to R12, R12 to R4, R6 to R5, R7 to R6, R8 to R7, R9 to R8, R10 to R9
Connections:
- net Analog10: now also Analog/GroundPins2.4 (Pin_4); no longer Analog/GroundPins1.10 (Pin_10)
- net Analog11: now also Analog/GroundPins2.6 (Pin_6); no longer Analog/GroundPins1.11 (Pin_11)
- net Analog12: now also Analog/GroundPins2.8 (Pin_8); no longer Analog/GroundPins1.12 (Pin_12)
- net Analog13: now also Analog/GroundPins2.10 (Pin_10); no longer Analog/GroundPins1.13 (Pin_13)
- net Analog14: now also Analog/GroundPins2.12 (Pin_12); no longer Analog/GroundPins1.14 (Pin_14)
- net Analog15: now also Analog/GroundPins2.14 (Pin_14); no longer Analog/GroundPins1.15 (Pin_15)
- net Analog2: now also Analog/GroundPins1.3 (Pin_3); no longer Analog/GroundPins1.2 (Pin_2)
- net Analog3: now also Analog/GroundPins1.5 (Pin_5); no longer Analog/GroundPins1.3 (Pin_3)
- net Analog4: now also Analog/GroundPins1.7 (Pin_7); no longer Analog/GroundPins1.4 (Pin_4)
- net Analog5: now also Analog/GroundPins1.9 (Pin_9); no longer Analog/GroundPins1.5 (Pin_5)
- net Analog6: now also Analog/GroundPins1.11 (Pin_11); no longer Analog/GroundPins1.6 (Pin_6)
- net Analog7: now also Analog/GroundPins1.13 (Pin_13); no longer Analog/GroundPins1.7 (Pin_7)
- net Analog8: now also Analog/GroundPins1.15 (Pin_15); no longer Analog/GroundPins1.8 (Pin_8)
- net Analog9: now also Analog/GroundPins2.2 (Pin_2); no longer Analog/GroundPins1.9 (Pin_9)
- net C1 discharge: now also Charge/DischargePins1.2 (Pin_2)
- net C10 charge: now also Charge/DischargePins2.4 (Pin_4); no longer Charge/DischargePins1.10 (Pin_10)
- net C10 discharge: now also Charge/DischargePins2.5 (Pin_5)
- net C11 charge: now also Charge/DischargePins2.6 (Pin_6); no longer Charge/DischargePins1.11 (Pin_11)
- net C11 discharge: now also Charge/DischargePins2.7 (Pin_7)
- net C12 charge: now also Charge/DischargePins2.8 (Pin_8); no longer Charge/DischargePins1.12 (Pin_12)
- net C12 discharge: now also Charge/DischargePins2.9 (Pin_9)
- net C13 charge: now also Charge/DischargePins2.10 (Pin_10); no longer Charge/DischargePins1.13 (Pin_13)
- net C13 discharge: now also Charge/DischargePins2.11 (Pin_11)
- net C14 charge: now also Charge/DischargePins2.12 (Pin_12); no longer Charge/DischargePins1.14 (Pin_14)
- net C14 discharge: now also Charge/DischargePins2.13 (Pin_13)
- net C15 charge: now also Charge/DischargePins2.14 (Pin_14); no longer Charge/DischargePins1.15 (Pin_15)
- net C15 discharge: now also Charge/DischargePins2.15 (Pin_15)
- net C2 charge: now also Charge/DischargePins1.3 (Pin_3); no longer Charge/DischargePins1.2 (Pin_2)
- net C2 discharge: now also Charge/DischargePins1.4 (Pin_4)
- net C3 charge: now also Charge/DischargePins1.5 (Pin_5); no longer Charge/DischargePins1.3 (Pin_3)
- net C3 discharge: now also Charge/DischargePins1.6 (Pin_6)
- net C4 charge: now also Charge/DischargePins1.7 (Pin_7); no longer Charge/DischargePins1.4 (Pin_4)
- net C4 discharge: now also Charge/DischargePins1.8 (Pin_8)
- net C5 charge: now also Charge/DischargePins1.9 (Pin_9); no longer Charge/DischargePins1.5 (Pin_5)
- net C5 discharge: now also Charge/DischargePins1.10 (Pin_10)
- net C6 charge: now also Charge/DischargePins1.11 (Pin_11); no longer Charge/DischargePins1.6 (Pin_6)
- net C6 discharge: now also Charge/DischargePins1.12 (Pin_12)
- net C7 charge: now also Charge/DischargePins1.13 (Pin_13); no longer Charge/DischargePins1.7 (Pin_7)
- net C7 discharge: now also Charge/DischargePins1.14 (Pin_14)
- net C8 charge: now also Charge/DischargePins1.15 (Pin_15); no longer Charge/DischargePins1.8 (Pin_8)
- net C8 discharge: now also Charge/DischargePins2.1 (Pin_1)
- net C9 charge: now also Charge/DischargePins2.2 (Pin_2); no longer Charge/DischargePins1.9 (Pin_9)
- net C9 discharge: now also Charge/DischargePins2.3 (Pin_3)
- net GND: now also Analog/GroundPins1.10 (Pin_10), Analog/GroundPins1.12 (Pin_12), Analog/GroundPins1.14 (Pin_14), Analog/GroundPins1.2 (Pin_2), Analog/GroundPins1.4 (Pin_4), Analog/GroundPins1.6 (Pin_6), Analog/GroundPins1.8 (Pin_8), Ground.1 (Pin_1); no longer Analog/GroundPins2.10 (Pin_10), Analog/GroundPins2.12 (Pin_12), Analog/GroundPins2.14 (Pin_14), Analog/GroundPins2.2 (Pin_2), Analog/GroundPins2.4 (Pin_4), Analog/GroundPins2.6 (Pin_6), Analog/GroundPins2.8 (Pin_8)
Other:
- moved on the sheet: Analog/GroundPins1

Commit message: Add files via upload
Parts:
- removed Charge/DischargePins1, Charge/DischargePins2: Conn_01x15_Female, Connector_PinHeader_2.54mm:PinHeader_1x15_P2.54mm_Vertical, symbol Connector:Conn_01x15_Female
- removed Ground: Conn_01x01_Female, Connector_PinHeader_2.54mm:PinHeader_1x01_P2.54mm_Vertical, symbol Connector:Conn_01x01_Female
- added Charge/DischargePins1: Conn_01x31_Female, Connector_PinHeader_2.54mm:PinHeader_1x31_P2.54mm_Vertical, symbol Connector:Conn_01x31_Female
Connections:
- net C1 charge: now also Charge/DischargePins1.2 (Pin_2)
- net C1 discharge: now also Charge/DischargePins1.3 (Pin_3)
- net C10 charge: now also Charge/DischargePins1.20 (Pin_20)
- net C10 discharge: now also Charge/DischargePins1.21 (Pin_21)
- net C11 charge: now also Charge/DischargePins1.22 (Pin_22)
- net C11 discharge: now also Charge/DischargePins1.23 (Pin_23)
- net C12 charge: now also Charge/DischargePins1.24 (Pin_24)
- net C12 discharge: now also Charge/DischargePins1.25 (Pin_25)
- net C13 charge: now also Charge/DischargePins1.26 (Pin_26)
- net C13 discharge: now also Charge/DischargePins1.27 (Pin_27)
- net C14 charge: now also Charge/DischargePins1.28 (Pin_28)
- net C14 discharge: now also Charge/DischargePins1.29 (Pin_29)
- net C15 charge: now also Charge/DischargePins1.30 (Pin_30)
- net C15 discharge: now also Charge/DischargePins1.31 (Pin_31)
- net C2 charge: now also Charge/DischargePins1.4 (Pin_4)
- net C2 discharge: now also Charge/DischargePins1.5 (Pin_5)
- net C3 charge: now also Charge/DischargePins1.6 (Pin_6)
- net C3 discharge: now also Charge/DischargePins1.7 (Pin_7)
- net C4 charge: now also Charge/DischargePins1.8 (Pin_8)
- net C4 discharge: now also Charge/DischargePins1.9 (Pin_9)
- net C5 charge: now also Charge/DischargePins1.10 (Pin_10)
- net C5 discharge: now also Charge/DischargePins1.11 (Pin_11)
- net C6 charge: now also Charge/DischargePins1.12 (Pin_12)
- net C6 discharge: now also Charge/DischargePins1.13 (Pin_13)
- net C7 charge: now also Charge/DischargePins1.14 (Pin_14)
- net C7 discharge: now also Charge/DischargePins1.15 (Pin_15)
- net C8 charge: now also Charge/DischargePins1.16 (Pin_16)
- net C8 discharge: now also Charge/DischargePins1.17 (Pin_17)
- net C9 charge: now also Charge/DischargePins1.18 (Pin_18)
- net C9 discharge: now also Charge/DischargePins1.19 (Pin_19)
- net GND: now also Charge/DischargePins1.1 (Pin_1)
