File: CapSensors.kicad_pcb (KiCad board)
At the start: 2 copper layers, 6 parts, among them J1 Charge/Discharge Pins, J2 Analog Pins, J3 Ground, J4 Charge/Discharge Pins

Commit message: Add files via upload
Parts:
- removed J1, J4: Charge/Discharge Pins, TerminalBlock_4Ucon:TerminalBlock_4Ucon_1x15_P3.50mm_Vertical
- removed J2: Analog Pins, TerminalBlock_4Ucon:TerminalBlock_4Ucon_1x15_P3.50mm_Vertical
- removed J3: Ground, TerminalBlock_4Ucon:TerminalBlock_4Ucon_1x15_P3.50mm_Vertical
- added AnalogPins1: Screw_Terminal_01x15, TerminalBlock_TE-Connectivity:TerminalBlock_TE_1-282834-2_1x12_P2.54mm_Horizontal, F.Cu at (189.3, 39.3)
- added ChargePins1: Conn_01x15_Male, Connector_PinHeader_2.54mm:PinHeader_1x15_P2.54mm_Vertical, F.Cu at (179.8, 28.8)
- added DischargePins1: Conn_01x15_Male, Connector_PinHeader_2.54mm:PinHeader_1x15_P2.54mm_Vertical, F.Cu at (184.4, 28.8)
- added Ground1: Screw_Terminal_01x15, TerminalBlock_TE-Connectivity:TerminalBlock_TE_1-282834-2_1x12_P2.54mm_Horizontal, F.Cu at (189.3, 30.8)
- added R10: 10k, Resistor_SMD:R_0603_1608Metric, F.Cu at (200.8, 49.9)
- added R11: 220, Resistor_SMD:R_0603_1608Metric, F.Cu at (196.8, 47.3)
- added R12: 220, Resistor_SMD:R_0603_1608Metric, F.Cu at (192.8, 47.3)
- added R13: 10k, Resistor_SMD:R_0603_1608Metric, F.Cu at (196.8, 52.4)
- added R14: 220, Resistor_SMD:R_0603_1608Metric, F.Cu at (204.8, 44.8)
- added R15: 10k, Resistor_SMD:R_0603_1608Metric, F.Cu at (179.5, 70.4)
- added R16: 220, Resistor_SMD:R_0603_1608Metric, F.Cu at (196.8, 49.9)
- added R17: 10k, Resistor_SMD:R_0603_1608Metric, F.Cu at (192.8, 57.4)
- added R18: 220, Resistor_SMD:R_0603_1608Metric, F.Cu at (188.8, 54.9)
- added R19: 10k, Resistor_SMD:R_0603_1608Metric, F.Cu at (196.8, 44.8)
- added R20: 220, Resistor_SMD:R_0603_1608Metric, F.Cu at (200.8, 47.3)
- added R21: 10k, Resistor_SMD:R_0603_1608Metric, F.Cu at (183.5, 67.9)
- added R22: 220, Resistor_SMD:R_0603_1608Metric, F.Cu at (192.8, 44.8)
- added R23: 10k, Resistor_SMD:R_0603_1608Metric, F.Cu at (200.8, 44.8)
- added R24: 220, Resistor_SMD:R_0603_1608Metric, F.Cu at (188.8, 47.3)
- added R25: 10k, Resistor_SMD:R_0603_1608Metric, F.Cu at (221.8, 27.7)
- added R26: 220, Resistor_SMD:R_0603_1608Metric, F.Cu at (192.8, 59.9)
- added R27: 10k, Resistor_SMD:R_0603_1608Metric, F.Cu at (188.8, 44.8)
- added R28: 220, Resistor_SMD:R_0603_1608Metric, F.Cu at (188.8, 49.9)
- added R29: 10k, Resistor_SMD:R_0603_1608Metric, F.Cu at (192.8, 54.9)
- added R3: 10k, Resistor_SMD:R_0603_1608Metric, F.Cu at (188.8, 62.4)
- added R30: 220, Resistor_SMD:R_0603_1608Metric, F.Cu at (221.8, 30.2)
- added R4: 10k, Resistor_SMD:R_0603_1608Metric, F.Cu at (192.8, 52.4)
- added R5: 220, Resistor_SMD:R_0603_1608Metric, F.Cu at (183.5, 70.4)
- added R6: 10k, Resistor_SMD:R_0603_1608Metric, F.Cu at (188.8, 59.9)
- added R7: 220, Resistor_SMD:R_0603_1608Metric, F.Cu at (188.8, 57.4)
- added R8: 10k, Resistor_SMD:R_0603_1608Metric, F.Cu at (225.8, 27.7)
- added R9: 220, Resistor_SMD:R_0603_1608Metric, F.Cu at (179.5, 67.9)
- moved R2 29.5 mm to (188.8, 52.4)
- moved R1 23.1 mm to (192.8, 49.9)
Connections:
- net Net-(R1-Pad2) renamed Analog1

Commit message: Add files via upload
Parts:
- AnalogPins1, Ground1: footprint TerminalBlock_TE-Connectivity:TerminalBlock_TE_1-282834-2_1x12_P2.54mm_Horizontal -> Connector_PinHeader_2.54mm:PinHeader_1x15_P2.54mm_Vertical
- ChargePins1, DischargePins1: value Conn_01x15_Male -> Conn_01x15_Female
- moved Ground1 68.9 mm to (120.5, 34.3)
- moved R8 57.2 mm to (172.2, 47.6)
- moved AnalogPins1 56.4 mm to (133.1, 34.0)
- moved R22 48.2 mm to (157.6, 77.7)
- moved R27 48.2 mm to (153.6, 77.7)
- moved R25 41.4 mm to (184.2, 45.1)
- moved DischargePins1 41.2 mm to (224.8, 37.2)
- moved R30 36.7 mm to (188.2, 45.1)
- moved ChargePins1 35.7 mm to (214.6, 36.9)
- moved R21 32.4 mm to (172.2, 37.5)
- moved R13 26.5 mm to (172.2, 42.5)
- moved R15 25.4 mm to (180.2, 45.1)
- moved R5 24.0 mm to (176.2, 47.6)
- moved R6 22.3 mm to (172.2, 45.1)
- moved R23 21.9 mm to (180.2, 37.5)
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Connections:
- ChargePins1 pad 10: unconnected-(ChargePins1-Pad10) -> C10 charge
- ChargePins1 pad 11: unconnected-(ChargePins1-Pad11) -> C11 charge
- ChargePins1 pad 12: unconnected-(ChargePins1-Pad12) -> C12 charge
- ChargePins1 pad 13: unconnected-(ChargePins1-Pad13) -> C13 charge
- ChargePins1 pad 14: unconnected-(ChargePins1-Pad14) -> C14 charge
- ChargePins1 pad 15: unconnected-(ChargePins1-Pad15) -> C15 charge
- ChargePins1 pad 2: unconnected-(ChargePins1-Pad2) -> C2 charge
- ChargePins1 pad 3: unconnected-(ChargePins1-Pad3) -> C3 charge
- ChargePins1 pad 4: unconnected-(ChargePins1-Pad4) -> C4 charge
- ChargePins1 pad 5: unconnected-(ChargePins1-Pad5) -> C5 charge
- ChargePins1 pad 6: unconnected-(ChargePins1-Pad6) -> C6 charge
- ChargePins1 pad 7: unconnected-(ChargePins1-Pad7) -> C7 charge
- ChargePins1 pad 8: unconnected-(ChargePins1-Pad8) -> C8 charge
- ChargePins1 pad 9: unconnected-(ChargePins1-Pad9) -> C9 charge
- DischargePins1 pad 10: unconnected-(DischargePins1-Pad10) -> C10 discharge
- DischargePins1 pad 11: unconnected-(DischargePins1-Pad11) -> C11 discharge
- DischargePins1 pad 12: unconnected-(DischargePins1-Pad12) -> C12 discharge
- DischargePins1 pad 13: unconnected-(DischargePins1-Pad13) -> C13 discharge
- DischargePins1 pad 14: unconnected-(DischargePins1-Pad14) -> C14 discharge
- DischargePins1 pad 15: unconnected-(DischargePins1-Pad15) -> C15 discharge
- DischargePins1 pad 2: unconnected-(DischargePins1-Pad2) -> C2 discharge
- DischargePins1 pad 3: unconnected-(DischargePins1-Pad3) -> C3 discharge
- DischargePins1 pad 4: unconnected-(DischargePins1-Pad4) -> C4 discharge
- DischargePins1 pad 5: unconnected-(DischargePins1-Pad5) -> C5 discharge
- DischargePins1 pad 6: unconnected-(DischargePins1-Pad6) -> C6 discharge
- DischargePins1 pad 7: unconnected-(DischargePins1-Pad7) -> C7 discharge
- DischargePins1 pad 8: unconnected-(DischargePins1-Pad8) -> C8 discharge
- DischargePins1 pad 9: unconnected-(DischargePins1-Pad9) -> C9 discharge

Commit message: Add files via upload
Parts:
- removed AnalogPins1, Ground1: Screw_Terminal_01x15, Connector_PinHeader_2.54mm:PinHeader_1x15_P2.54mm_Vertical
- removed ChargePins1, DischargePins1: Conn_01x15_Female, Connector_PinHeader_2.54mm:PinHeader_1x15_P2.54mm_Vertical
- added Analog/GroundPins1: Screw_Terminal_01x15, Connector_PinHeader_2.54mm:PinHeader_1x15_P2.54mm_Vertical, F.Cu at (121.6, 81.3)
- added Analog/GroundPins2: Screw_Terminal_01x15, Connector_PinHeader_2.54mm:PinHeader_1x15_P2.54mm_Vertical, F.Cu at (121.6, 120.5)
- added Charge/DischargePins1: Conn_01x15_Female, Connector_PinHeader_2.54mm:PinHeader_1x15_P2.54mm_Vertical, F.Cu at (134.2, 81.1)
- added Charge/DischargePins2: Conn_01x15_Female, Connector_PinHeader_2.54mm:PinHeader_1x15_P2.54mm_Vertical, F.Cu at (134.2, 120.2)
- added GND: Conn_01x01_Female, Connector_PinHeader_2.54mm:PinHeader_1x01_P2.54mm_Vertical, F.Cu at (130.9, 159.4)
- added REF**: MountingHole_2.1mm, MountingHole:MountingHole_2.1mm, F.Cu at (136.6, 160.4)
- added REF**: MountingHole_2.1mm, MountingHole:MountingHole_2.1mm, F.Cu at (120.0, 76.1)
- R10, R4, R6, R8: value 10k -> 220
- R11, R5, R7, R9: value 220 -> 10k
- moved R28 131.0 mm to (128.4, 149.6)
- moved R30 124.6 mm to (128.5, 154.4)
- moved R29 121.4 mm to (128.5, 152.4), turned to 180 degrees
- moved R24 112.6 mm to (128.3, 139.4)
- moved R23 112.2 mm to (128.3, 137.0), turned to 180 degrees
- moved R25 111.9 mm to (128.4, 142.1), turned to 180 degrees
- moved R26 111.8 mm to (128.4, 144.5)
- moved R20 111.8 mm to (128.3, 129.3)
- moved R21 104.0 mm to (128.3, 131.8), turned to 180 degrees
- moved R17 101.7 mm to (128.4, 121.7), turned to 180 degrees
- moved R19 99.0 mm to (128.3, 126.7), turned to 180 degrees
- moved R16 96.8 mm to (128.3, 119.0)
- moved R18 94.6 mm to (128.4, 124.2)
- moved R14 93.8 mm to (128.3, 112.8)
- moved R11 90.5 mm to (128.3, 105.4), turned to 180 degrees
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Connections:
- R10 pad 1: C5 charge -> Analog5
- R10 pad 2: Analog5 -> C5 discharge
- R11 pad 1: Analog5 -> C6 charge
- R11 pad 2: C5 discharge -> Analog6
- R12 pad 1: Analog2 -> Analog6
- R12 pad 2: C2 discharge -> C6 discharge
- R4 pad 1: C6 charge -> Analog2
- R4 pad 2: Analog6 -> C2 discharge
- R5 pad 1: Analog6 -> C3 charge
- R5 pad 2: C6 discharge -> Analog3
- R6 pad 1: C3 charge -> Analog3
- R6 pad 2: Analog3 -> C3 discharge
- R7 pad 1: Analog3 -> C4 charge
- R7 pad 2: C3 discharge -> Analog4
- R8 pad 1: C4 charge -> Analog4
- R8 pad 2: Analog4 -> C4 discharge
- R9 pad 1: Analog4 -> C5 charge
- R9 pad 2: C4 discharge -> Analog5
Routing:
- net GND: track 0.00 -> 56.7 mm, vias 0 -> 16
- net Analog8: track 0.00 -> 9.29 mm
- net Analog11: track 0.00 -> 8.59 mm
- net Analog14: track 0.00 -> 8.56 mm
- net Analog10: track 0.00 -> 8.51 mm
- net Analog9: track 0.00 -> 8.49 mm
- net Analog13: track 0.00 -> 8.47 mm
- net Analog5: track 0.00 -> 8.39 mm
- net Analog12: track 0.00 -> 8.35 mm
- net Analog6: track 0.00 -> 8.32 mm
- net Analog7: track 0.00 -> 8.31 mm
- net Analog4: track 0.00 -> 8.23 mm
- net Analog15: track 0.00 -> 8.14 mm
- net Analog3: track 0.00 -> 8.12 mm
- net Analog2: track 0.00 -> 7.87 mm
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- added copper zone on B.Cu, net GND
Other:
- board outline added: 23.1 x 90.9 mm
- board text added: "A1"
- board text added: "A10"
- board text added: "A11"
- board text added: "A12"
- board text added: "A13"
- board text added: "A14"
- board text added: "A15"
- board text added: "A2"
- board text added: "A3"
- board text added: "A4"
- board text added: "A5"
- board text added: "A6"
- board text added: "A7"
- board text added: "A8"
- board text added: "A9"
- board text added: "C1"
- board text added: "C10"
- board text added: "C11"
- board text added: "C12"
- board text added: "C13"
- board text added: "C14"
- board text added: "C15"
- board text added: "C2"
- board text added: "C3"
- board text added: "C4"
- board text added: "C5"
- board text added: "C6"
- board text added: "C7"
- board text added: "C8"
- board text added: "C9"
- board text added: "D1"
- board text added: "D10"
- board text added: "D11"
- board text added: "D12"
- board text added: "D13"
- board text added: "D14"
- board text added: "D15"
- board text added: "D2"
- board text added: "D3"
- board text added: "D4"
- board text added: "D5"
- board text added: "D6"
- board text added: "D7"
- board text added: "D8"
- board text added: "D9"
- board text added: "GND"
- board text added: "Jumbo Animal I Spy Sensor Board"
- board text added: "Team Kablooey"

Commit message: Add files via upload
Parts:
- removed Charge/DischargePins2: Conn_01x15_Female, Connector_PinHeader_2.54mm:PinHeader_1x15_P2.54mm_Vertical
- removed GND: Conn_01x01_Female, Connector_PinHeader_2.54mm:PinHeader_1x01_P2.54mm_Vertical
- Charge/DischargePins1: value Conn_01x15_Female -> Conn_01x31_Female; footprint Connector_PinHeader_2.54mm:PinHeader_1x15_P2.54mm_Vertical -> Connector_PinHeader_2.54mm:PinHeader_1x31_P2.54mm_Vertical
- moved Charge/DischargePins1 2.64 mm to (134.2, 78.5)
- moved REF** 0.81 mm to (136.5, 159.6)
Connections:
- Charge/DischargePins1 pad 1: C1 charge -> GND
- Charge/DischargePins1 pad 10: C5 discharge -> C5 charge
- Charge/DischargePins1 pad 11: C6 charge -> C5 discharge
- Charge/DischargePins1 pad 12: C6 discharge -> C6 charge
- Charge/DischargePins1 pad 13: C7 charge -> C6 discharge
- Charge/DischargePins1 pad 14: C7 discharge -> C7 charge
- Charge/DischargePins1 pad 15: C8 charge -> C7 discharge
- Charge/DischargePins1 pad 2: C1 discharge -> C1 charge
- Charge/DischargePins1 pad 3: C2 charge -> C1 discharge
- Charge/DischargePins1 pad 4: C2 discharge -> C2 charge
- Charge/DischargePins1 pad 5: C3 charge -> C2 discharge
- Charge/DischargePins1 pad 6: C3 discharge -> C3 charge
- Charge/DischargePins1 pad 7: C4 charge -> C3 discharge
- Charge/DischargePins1 pad 8: C4 discharge -> C4 charge
- Charge/DischargePins1 pad 9: C5 charge -> C4 discharge
Routing:
- net GND: track 56.7 -> 61.6 mm
Other:
- board size 23.1 x 90.9 mm -> 23.1 x 90.2 mm

Commit message: Add files via upload
Parts:
- added Analogs1: Conn_01x15_Female, Connector_PinHeader_2.54mm:PinHeader_1x15_P2.54mm_Vertical, F.Cu at (141.3, 98.6)
- moved REF** 8.30 mm to (143.2, 154.7)
Routing:
- net Analog15: track 8.14 -> 37.7 mm
- net Analog1: track 7.80 -> 34.5 mm
- net Analog14: track 8.56 -> 35.0 mm
- net Analog2: track 7.87 -> 32.2 mm
- net Analog3: track 8.12 -> 32.1 mm
- net Analog13: track 8.47 -> 32.4 mm
- net Analog12: track 8.35 -> 29.8 mm
- net Analog4: track 8.23 -> 28.6 mm
- net Analog11: track 8.59 -> 28.1 mm
- net Analog5: track 8.39 -> 25.3 mm
- net Analog10: track 8.51 -> 25.1 mm
- net Analog6: track 8.32 -> 24.0 mm
- net Analog9: track 8.49 -> 23.9 mm
- net Analog7: track 8.31 -> 23.2 mm
- net Analog8: track 9.29 -> 24.0 mm
Other:
- board size 23.1 x 90.2 mm -> 30.2 x 86.4 mm
